Commit message: Motion simulation confirmed

File: urdf/armed3w.gazebo.xacro (robot description, xacro)
@@ -1,4 +1,5 @@
 <?xml version="1.0" encoding="UTF-8"?>
 <robot name="armed3w" xmlns:xacro="http://ros.org/wiki/xacro">
+  <xacro:property name="pi" value="3.1415926" />
   <!-- coefficient of friction start-->
   <gazebo reference="body">
@@ -72,9 +73,9 @@
       <pose>0 0 0 0 0 0</pose>
       <visualize>true</visualize>
-      <update_rate>2</update_rate>
+      <update_rate>20</update_rate>
       <ray>
         <scan>
           <horizontal>
-            <samples>21</samples>
+            <samples>101</samples>
             <resolution>1</resolution>
             <min_angle>-3.1415926</min_angle>

Commit message: Tuning is over with bb8

File: urdf/armed3w.gazebo.xacro (robot description, xacro)
@@ -5,31 +5,31 @@
   <gazebo reference="body">
     <selfCollide>true</selfCollide>
-      <mu1 value="0.05"/>
-      <mu2 value="0.05"/>
+    <mu1 value="0.05"/>
+    <mu2 value="0.05"/>
   </gazebo>
   <gazebo reference="wheelFront">
     <selfCollide>true</selfCollide>
-      <mu1 value="0.0"/>
-      <mu2 value="0.0"/>
+    <mu1 value="0.0"/>
+    <mu2 value="0.0"/>
   </gazebo>
   <gazebo reference="wheelRight">
     <selfCollide>true</selfCollide>
-      <mu1 value="0.8"/>
-      <mu2 value="0.8"/>
+    <mu1 value="0.8"/>
+    <mu2 value="0.8"/>
   </gazebo>
   <gazebo reference="wheelLeft">
     <selfCollide>true</selfCollide>
-      <mu1 value="0.8"/>
-      <mu2 value="0.8"/>
+    <mu1 value="0.8"/>
+    <mu2 value="0.8"/>
   </gazebo>
   <gazebo reference="armRight">
     <selfCollide>true</selfCollide>
-      <mu1 value="0.8"/>
-      <mu2 value="0.8"/>
+    <mu1 value="0.8"/>
+    <mu2 value="0.8"/>
   </gazebo>
   <gazebo reference="armLeft">
     <selfCollide>true</selfCollide>
-      <mu1 value="0.8"/>
-      <mu2 value="0.8"/>
+    <mu1 value="0.8"/>
+    <mu2 value="0.8"/>
   </gazebo>
   <!-- coefficient of friction end-->
@@ -72,10 +72,10 @@
     <sensor type="ray" name="lds_lfcd_sensor">
       <pose>0 0 0 0 0 0</pose>
-      <visualize>true</visualize>
-      <update_rate>20</update_rate>
+      <visualize>false</visualize>
+      <update_rate>50</update_rate>
       <ray>
         <scan>
           <horizontal>
-            <samples>101</samples>
+            <samples>51</samples>
             <resolution>1</resolution>
             <min_angle>-3.1415926</min_angle>

File: urdf/armed3w_bb8.urdf.xacro (robot description, xacro)
@@ -4,5 +4,4 @@
   <xacro:property name="body_height" value="0.4" />
   <xacro:property name="wheel_radius" value="0.05" />
-  <xacro:property name="arm_length" value="0.6" />
   <xacro:property name="pi" value="3.1415926" />
   <xacro:property name="sensor_size" value=".1" />
@@ -17,6 +16,6 @@
     <inertial>
       <mass value="1"/>
-      <!-- #cylinder Izz = 1/2 * M * r^2 -->
-      <!-- #cylinder Iyy = Ixx = 1/12 * M * l^2 -->
+      #cylinder Izz = 1/2 * M * r^2
+      #cylinder Iyy = Ixx = 1/12 * M * l^2
       <inertia ixx=".0675"  ixy="0"  ixz="0" iyy=".0675" iyz="0" izz=".045"/>
     </inertial>
@@ -27,8 +26,8 @@
       </geometry>
     </collision>
-    <visual>
-      <origin xyz="0 0 0" rpy="0 0 0"/>
+    <visual name='bb8_visual'>
+      <origin xyz="0 0 -.26" rpy="0 0 0"/>
       <geometry>
-        <cylinder radius=".3" length="${body_height}"/>
+        <mesh filename="package://robot_utokyo/models/bb8/meshes/BB8.dae" scale=".05 .05 .05"/>
       </geometry>
     </visual>
@@ -54,5 +53,5 @@
       <origin xyz="0 0 0" rpy="0 0 0"/>
       <geometry>
-        <sphere radius="${wheel_radius}"/>
+        <sphere radius=".001"/>
       </geometry>
     </visual>
@@ -79,5 +78,5 @@
       <origin xyz="0 0 0" rpy="0 0 0"/>
       <geometry>
-        <sphere radius="${wheel_radius}"/>
+        <sphere radius=".001"/>
       </geometry>
     </visual>
@@ -104,60 +103,8 @@
       <origin xyz="0 0 0" rpy="0 0 0"/>
       <geometry>
-        <sphere radius="${wheel_radius}"/>
+        <sphere radius=".001"/>
       </geometry>
     </visual>
   </link>
-  <joint name="body_armRight" type="continuous">
-    <parent link="body"/>
-    <child link="armRight"/>
-    <origin xyz=".3 0 .2" rpy="${- pi / 2} 0 0"/>
-    <axis xyz="1 0 0"/>
-  </joint>
-  <link name='armRight'>
-    <inertial>
-      <mass value=".1"/>
-      <!-- #cylinder Izz = 1/2 * M * r^2 -->
-      <!-- #cylinder Iyy = Ixx = 1/12 * M * l^2 -->
-      <inertia ixx=".003"  ixy="0"  ixz="0" iyy=".003" iyz="0" izz=".000045"/>
-    </inertial>
-    <collision>
-      <origin xyz="0 0 -.3" rpy="0 0 0"/>
-      <geometry>
-        <cylinder radius=".03" length="${arm_length}"/>
-      </geometry>
-    </collision>
-    <visual>
-      <origin xyz="0 0 -.3" rpy="0 0 0"/>
-      <geometry>
-        <cylinder radius=".03" length="${arm_length}"/>
-      </geometry>
-    </visual>
-  </link>
-  <joint name="body_armLeft" type="continuous">
-    <parent link="body"/>
-    <child link="armLeft"/>
-    <origin xyz="-.3 0 .2" rpy="${- pi / 2} 0 0"/>
-    <axis xyz="1 0 0"/>
-  </joint>
-  <link name='armLeft'>
-      <inertial>
-        <mass value=".1"/>
-      <!-- #cylinder Izz = 1/2 * M * r^2
-      #cylinder Iyy = Ixx = 1/12 * M * l^2 -->
-      <inertia ixx=".003"  ixy="0"  ixz="0" iyy=".003" iyz="0" izz=".000045"/>
-      </inertial>
-      <collision>
-        <origin xyz="0 0 -.3" rpy="0 0 0"/>
-        <geometry>
-          <cylinder radius=".03" length="${arm_length}"/>
-        </geometry>
-      </collision>
-      <visual>
-        <origin xyz="0 0 -.3" rpy="0 0 0"/>
-        <geometry>
-          <cylinder radius=".03" length="${arm_length}"/>
-        </geometry>
-      </visual>
-    </link>
   <!-- controller start-->
   <transmission name="body_wheelRight_trans">
@@ -177,24 +124,4 @@
     </joint>
     <actuator name="body_wheelLeft_motor">
-      <hardwareInterface>VelocityJointInterface</hardwareInterface>
-      <mechanicalReduction>30</mechanicalReduction>
-    </actuator>
-  </transmission>
-  <transmission name="body_armRight_trans">
-    <type>transmission_interface/SimpleTransmission</type>
-    <joint name="body_armRight">
-      <hardwareInterface>hardware_interface/VelocityJointInterface</hardwareInterface>
-    </joint>
-    <actuator name="body_armRight_motor">
-      <hardwareInterface>VelocityJointInterface</hardwareInterface>
-      <mechanicalReduction>30</mechanicalReduction>
-    </actuator>
-  </transmission>
-  <transmission name="body_armLeft_trans">
-    <type>transmission_interface/SimpleTransmission</type>
-    <joint name="body_armLeft">
-      <hardwareInterface>hardware_interface/VelocityJointInterface</hardwareInterface>
-    </joint>
-    <actuator name="body_armLeft_motor">
       <hardwareInterface>VelocityJointInterface</hardwareInterface>
       <mechanicalReduction>30</mechanicalReduction>
