Commit message: add sensor, but rviz failed

File: urdf/armed3w.urdf (robot description, URDF)
Before this commit: robot armed3w, 7 links, 6 joints
Joints:
- joint base_link_joint: origin xyz=0 0 0 -> xyz=-4 5 0
- joint body_wheelFront: axis 1 0 0 -> (none)

Commit message: sensor added

File: urdf/armed3w.urdf (robot description, URDF)
Before this commit: robot armed3w, 7 links, 6 joints
Links:
- added link pico_flexx_depth_frame
- added link pico_flexx_link, mass 1; collision box size=0.007 0.066 0.016; visual box size=0.007 0.066 0.016
- added link pico_flexx_link_optical_frame
Joints:
- added joint pico_flexx_base_joint: type fixed, parent body, child pico_flexx_link_optical_frame, origin xyz=0.3 0 0.07 rpy=0 0 0
- added joint pico_flexx_depth_joint: type fixed, parent pico_flexx_link_optical_frame, child pico_flexx_depth_frame, origin xyz=0 0 0 rpy=${-M_PI/2} 0 ${-M_PI/2}
- added joint pico_flexx_joint: type fixed, parent pico_flexx_link_optical_frame, child pico_flexx_link, origin xyz=0 0 0 rpy=0 0 0
- joint body_armLeft: axis 1 0 0 -> 0 1 0; origin xyz=-.3 0 .2 rpy=0 0 0 -> xyz=0 -.3 .2 rpy=0 0 0
- joint body_armRight: axis 1 0 0 -> 0 1 0; origin xyz=.3 0 .2 rpy=0 0 0 -> xyz=0 .3 .2 rpy=0 0 0
- joint body_wheelFront: axis 1 0 0 -> (none); origin xyz=0 .2 -.48 rpy=0 0 0 -> xyz=.2 0 -.48 rpy=0 0 0
- joint body_wheelLeft: axis 1 0 0 -> 0 1 0; origin xyz=-0.1732 -.1 -.48 rpy=0 0 0 -> xyz=-.1 -0.1732 -.48 rpy=0 0 0
- joint body_wheelRight: axis 1 0 0 -> 0 1 0; origin xyz=0.1732 -.1 -.48 rpy=0 0 0 -> xyz=-.1 0.1732 -.48 rpy=0 0 0

Commit message: final source

File: urdf/armed3w.urdf (robot description, URDF)
Before this commit: robot armed3w, 9 links, 8 joints
Links:
- added link stopper1, mass 0; collision cylinder length=.01 radius=.02; visual cylinder length=.01 radius=.02
- added link stopper2, mass 0; collision cylinder length=.01 radius=.02; visual cylinder length=.01 radius=.02
- added link stopper3, mass 0; collision cylinder length=.01 radius=.02; visual cylinder length=.01 radius=.02
- added link stopper4, mass 0; collision cylinder length=.01 radius=.02; visual cylinder length=.01 radius=.02
Joints:
- added joint body_stopper1: type fixed, parent body, child stopper1, origin xyz=0 -.275 .45 rpy=0 0 0
- added joint body_stopper2: type fixed, parent body, child stopper2, origin xyz=0  .275 .45 rpy=0 0 0
- added joint body_stopper3: type fixed, parent body, child stopper3, origin xyz= .275 0 .45 rpy=0 0 0
- added joint body_stopper4: type fixed, parent body, child stopper4, origin xyz=-.275 0 .45 rpy=0 0 0
- joint camera_joint: origin xyz=0 -.3 0 rpy=0 0 0 -> xyz=0 -.3 0 rpy=0 0  -1.570796
